File: blinCAN.kicad_pcb (KiCad board)
At the start: 2 copper layers, 127.1 x 67.1 mm, 95 parts, among them IC201 ATMEGA328P-AU, J501 Conn_Address, P101 Conn_PWR_IN, P102 Conn_PWR_IN, P103 CONN_ICSP, P104 USB B, P105 Conn_CAN, P106 Conn_CAN, P601 D-SUB 25, P602 D-SUB 25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

Commit message: Fix some silkscreen misplacements.
Other:
- board text added: "v0.1 2018 metalhead777"
- board text removed: "v0.1 2017 metalhead777"
Changed lines of the file:
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@@
-(kicad_pcb (version 4) (host pcbnew 4.0.7-e2-6376~58~ubuntu16.04.1)
+(kicad_pcb (version 4) (host pcbnew 4.0.7)
   (general
-    (links 0)
+    (links 270)
     (no_connects 1)
     (area 31.700399 46.406999 158.952001 113.663801)
     (thickness 1.6)
-    (drawings 55)
+    (drawings 58)
     (tracks 816)
     (zones 0)
@@
     (tags "capacitor 0603")
     (attr smd)
-    (fp_text reference C202 (at 0 1.25 270) (layer B.SilkS)
+    (fp_text reference C202 (at 0 1.3462 270) (layer B.SilkS)
       (effects (font (size 1 1) (thickness 0.15)) (justify mirror))
     )
@@
     (tags "capacitor 0603")
     (attr smd)
-    (fp_text reference C204 (at -0.9652 -1.651 180) (layer B.SilkS)
+    (fp_text reference C204 (at 4.064 -0.127 180) (layer B.SilkS)
       (effects (font (size 1 1) (thickness 0.15)) (justify mirror))
     )
@@
     (tags "capacitor 0603")
     (attr smd)
-    (fp_text reference C205 (at -0.508 1.4478 180) (layer B.SilkS)
+    (fp_text reference C205 (at 4.064 0.127 180) (layer B.SilkS)
       (effects (font (size 1 1) (thickness 0.15)) (justify mirror))
     )
@@
     (tags "capacitor 0603")
     (attr smd)
-    (fp_text reference C304 (at 0 1.5875 270) (layer B.SilkS)
+    (fp_text reference C304 (at 0.8636 1.6256 270) (layer B.SilkS)
       (effects (font (size 1 1) (thickness 0.15)) (justify mirror))
     )
@@
     (tags "capacitor 0603")
     (attr smd)
-    (fp_text reference C104 (at -0.9144 1.2954 270) (layer F.SilkS)
+    (fp_text reference C104 (at -1.778 1.3716 270) (layer F.SilkS)
       (effects (font (size 1 1) (thickness 0.15)))
     )
@@
     (tags "Diode MELF Handsoldering")
     (attr smd)
-    (fp_text reference D104 (at 0 -2.54 180) (layer B.SilkS)
+    (fp_text reference D104 (at -7.493 0.4318 180) (layer B.SilkS)
       (effects (font (size 1 1) (thickness 0.15)) (justify mirror))
     )
@@
     (descr "CP, Radial series, Radial, pin pitch=2.00mm, , diameter=5mm, Electrolytic Capacitor")
     (tags "CP Radial series Radial pin pitch 2.00mm  diameter 5mm Electrolytic Capacitor")
-    (fp_text reference C201 (at 1 -3.81) (layer F.SilkS)
+    (fp_text reference C201 (at -3.048 0.0254 90) (layer F.SilkS)
       (effects (font (size 1 1) (thickness 0.15)))
     )
@@
     (tags "resistor 0805")
     (attr smd)
-    (fp_text reference FB101 (at 0 2.1 180) (layer B.SilkS)
+    (fp_text reference FB101 (at -0.0254 1.7272 180) (layer B.SilkS)
       (effects (font (size 1 1) (thickness 0.15)) (justify mirror))
     )
@@
     (tags "resistor 0805")
     (attr smd)
-    (fp_text reference FB401 (at 0 2.1 180) (layer B.SilkS)
+    (fp_text reference FB401 (at -4.7498 0.6096 180) (layer B.SilkS)
       (effects (font (size 1 1) (thickness 0.15)) (justify mirror))
     )
@@
     (descr "USB B connector")
     (tags "USB_B USB_DEV")
-    (fp_text reference P104 (at 11.05 1.27 270) (layer F.SilkS)
+    (fp_text reference P104 (at 4.5212 10.0076 360) (layer F.SilkS)
       (effects (font (size 1 1) (thickness 0.15)))
     )
@@
     (descr "Resistor, Axial_DIN0207 series, Axial, Horizontal, pin pitch=10.16mm, 0.25W = 1/4W, length*diameter=6.3*2.5mm^2, http://cdn-reichelt.de/documents/datenblatt/B400/1_4W%23YAG.pdf")
     (tags "Resistor Axial_DIN0207 series Axial Horizontal pin pitch 10.16mm 0.25W = 1/4W length 6.3mm diameter 2.5mm")
-    (fp_text reference R103 (at 5.08 -2.31 90) (layer F.SilkS)
+    (fp_text reference R103 (at -2.2098 -0.4318 180) (layer F.SilkS)
       (effects (font (size 1 1) (thickness 0.15)))
     )
@@
     (tags "Mesurement Point Round Trough Hole 1.5mm Drill 0.8mm")
     (attr virtual)
-    (fp_text reference TP602 (at 0 -2) (layer F.SilkS)
+    (fp_text reference TP602 (at -3.556 0) (layer F.SilkS)
       (effects (font (size 1 1) (thickness 0.15)))
     )
@@
     (tags "Mesurement Point Round Trough Hole 1.5mm Drill 0.8mm")
     (attr virtual)
-    (fp_text reference TP603 (at 0 -2) (layer F.SilkS)
+    (fp_text reference TP603 (at -3.5052 -0.0254) (layer F.SilkS)
       (effects (font (size 1 1) (thickness 0.15)))
     )
@@
     (tags "Mesurement Point Round Trough Hole 1.5mm Drill 0.8mm")
     (attr virtual)
-    (fp_text reference TP604 (at 0 -2) (layer F.SilkS)
+    (fp_text reference TP604 (at -3.556 0) (layer F.SilkS)
       (effects (font (size 1 1) (thickness 0.15)))
     )
@@
     (tags "Mesurement Point Round Trough Hole 1.5mm Drill 0.8mm")
     (attr virtual)
-    (fp_text reference TP605 (at 0 -2) (layer F.SilkS)
+    (fp_text reference TP605 (at -3.556 0) (layer F.SilkS)
       (effects (font (size 1 1) (thickness 0.15)))
     )
@@
     (tags "CMS SOT")
     (attr smd)
-    (fp_text reference U101 (at 0 4.5) (layer B.SilkS)
+    (fp_text reference U101 (at 5.5118 -0.0254 90) (layer B.SilkS)
       (effects (font (size 1 1) (thickness 0.15)) (justify mirror))
     )
@@
     (tags "SSOP 0.65 PowerPAD")
     (attr smd)
-    (fp_text reference U601 (at 0 -6.55 90) (layer F.SilkS)
+    (fp_text reference U601 (at -5.4864 -5.1562 180) (layer F.SilkS)
       (effects (font (size 1 1) (thickness 0.15)))
     )
@@
     (pad 1 np_thru_hole circle (at 0 0) (size 3.2 3.2) (drill 3.2) (layers *.Cu *.Mask))
   )
+  (gr_line (start 78.105 57.0484) (end 77.47 57.0484) (layer F.SilkS) (width 0.15))
+  (gr_line (start 78.105 59.182) (end 78.105 57.0484) (layer F.SilkS) (width 0.15))
+  (gr_line (start 77.47 59.182) (end 78.105 59.182) (layer F.SilkS) (width 0.15))
   (gr_text github.com/metalhead777/blinCAN (at 82.169 104.902) (layer B.SilkS)
     (effects (font (size 1.5 1.5) (thickness 0.3)) (justify mirror))
@@
     (effects (font (size 3.5 3) (thickness 0.6)) (justify right))
   )
-  (gr_text "v0.1 2017\nmetalhead777" (at 82.423 101.854) (layer F.SilkS)
+  (gr_text "v0.1 2018\nmetalhead777" (at 82.423 101.854) (layer F.SilkS)
     (effects (font (size 1.5 1.5) (thickness 0.3)) (justify right))
   )

Commit message: Add fiducial marks
Parts:
- added REF**: Fiducial_1mm_Dia_2.54mm_Outer_CopperBottom, Fiducials:Fiducial_1mm_Dia_2.54mm_Outer_CopperBottom, F.Cu at (41.5, 109.7)
- added REF**: Fiducial_1mm_Dia_2.54mm_Outer_CopperBottom, Fiducials:Fiducial_1mm_Dia_2.54mm_Outer_CopperBottom, F.Cu at (155.8, 110.5)
- added REF**: Fiducial_1mm_Dia_2.54mm_Outer_CopperBottom, Fiducials:Fiducial_1mm_Dia_2.54mm_Outer_CopperBottom, F.Cu at (155.8, 49.5)
- added REF**: Fiducial_1mm_Dia_2.54mm_Outer_CopperTop, Fiducials:Fiducial_1mm_Dia_2.54mm_Outer_CopperTop, F.Cu at (155.8, 110.5)
- added REF**: Fiducial_1mm_Dia_2.54mm_Outer_CopperTop, Fiducials:Fiducial_1mm_Dia_2.54mm_Outer_CopperTop, F.Cu at (155.8, 49.5)
- added REF**: Fiducial_1mm_Dia_2.54mm_Outer_CopperTop, Fiducials:Fiducial_1mm_Dia_2.54mm_Outer_CopperTop, F.Cu at (54.2, 50.3)
- added REF**: Fiducial_1mm_Dia_2.54mm_Outer_CopperTop, Fiducials:Fiducial_1mm_Dia_2.54mm_Outer_CopperTop, F.Cu at (54.2, 109.7)
- added REF**: Fiducial_1mm_Dia_2.54mm_Outer_CopperBottom, Fiducials:Fiducial_1mm_Dia_2.54mm_Outer_CopperBottom, F.Cu at (41.5, 50.3)
Changed lines of the file:
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@@
 (kicad_pcb (version 4) (host pcbnew 4.0.7)
   (general
-    (links 270)
+    (links 0)
     (no_connects 1)
     (area 31.700399 46.406999 158.952001 113.663801)
@@
     (tracks 816)
     (zones 0)
-    (modules 95)
+    (modules 103)
     (nets 108)
   )
@@
     (pad 1 np_thru_hole circle (at 0 0) (size 3.2 3.2) (drill 3.2) (layers *.Cu *.Mask))
   )
+  (module Fiducials:Fiducial_1mm_Dia_2.54mm_Outer_CopperTop (layer F.Cu)
+    (at 155.829 110.49)
+    (descr "Circular Fiducial, 1mm bare copper top; 2.54mm keepout")
+    (tags marker)
+    (attr virtual)
+    (fp_text reference REF** (at 3.048 2.794) (layer F.SilkS) hide
+      (effects (font (size 1 1) (thickness 0.15)))
+    )
+    (fp_text value Fiducial_1mm_Dia_2.54mm_Outer_CopperTop (at 0 -1.8) (layer F.Fab)
+      (effects (font (size 1 1) (thickness 0.15)))
+    )
+    (fp_circle (center 0 0) (end 1.55 0) (layer F.CrtYd) (width 0.05))
+    (pad ~ smd circle (at 0 0) (size 1 1) (layers F.Cu F.Mask)
+      (solder_mask_margin 0.77) (clearance 0.77))
+  )
+  (module Fiducials:Fiducial_1mm_Dia_2.54mm_Outer_CopperTop (layer F.Cu)
+    (at 155.829 49.53)
+    (descr "Circular Fiducial, 1mm bare copper top; 2.54mm keepout")
+    (tags marker)
+    (attr virtual)
+    (fp_text reference REF** (at 3.4 0.7) (layer F.SilkS) hide
+      (effects (font (size 1 1) (thickness 0.15)))
+    )
+    (fp_text value Fiducial_1mm_Dia_2.54mm_Outer_CopperTop (at 0 -1.8) (layer F.Fab)
+      (effects (font (size 1 1) (thickness 0.15)))
+    )
+    (fp_circle (center 0 0) (end 1.55 0) (layer F.CrtYd) (width 0.05))
+    (pad ~ smd circle (at 0 0) (size 1 1) (layers F.Cu F.Mask)
+      (solder_mask_margin 0.77) (clearance 0.77))
+  )
+  (module Fiducials:Fiducial_1mm_Dia_2.54mm_Outer_CopperTop (layer F.Cu)
+    (at 54.229 50.292)
+    (descr "Circular Fiducial, 1mm bare copper top; 2.54mm keepout")
+    (tags marker)
+    (attr virtual)
+    (fp_text reference REF** (at 3.4 0.7) (layer F.SilkS) hide
+      (effects (font (size 1 1) (thickness 0.15)))
+    )
+    (fp_text value Fiducial_1mm_Dia_2.54mm_Outer_CopperTop (at 0 -1.8) (layer F.Fab)
+      (effects (font (size 1 1) (thickness 0.15)))
+    )
+    (fp_circle (center 0 0) (end 1.55 0) (layer F.CrtYd) (width 0.05))
+    (pad ~ smd circle (at 0 0) (size 1 1) (layers F.Cu F.Mask)
+      (solder_mask_margin 0.77) (clearance 0.77))
+  )
+  (module Fiducials:Fiducial_1mm_Dia_2.54mm_Outer_CopperTop (layer F.Cu)
+    (at 54.229 109.728)
+    (descr "Circular Fiducial, 1mm bare copper top; 2.54mm keepout")
+    (tags marker)
+    (attr virtual)
+    (fp_text reference REF** (at 3.4 0.7) (layer F.SilkS) hide
+      (effects (font (size 1 1) (thickness 0.15)))
+    )
+    (fp_text value Fiducial_1mm_Dia_2.54mm_Outer_CopperTop (at 0 -1.8) (layer F.Fab)
+      (effects (font (size 1 1) (thickness 0.15)))
+    )
+    (fp_circle (center 0 0) (end 1.55 0) (layer F.CrtYd) (width 0.05))
+    (pad ~ smd circle (at 0 0) (size 1 1) (layers F.Cu F.Mask)
+      (solder_mask_margin 0.77) (clearance 0.77))
+  )
+  (module Fiducials:Fiducial_1mm_Dia_2.54mm_Outer_CopperBottom (layer F.Cu)
+    (at 41.529 50.292)
+    (descr "Circular Fiducial, 1mm bare copper bottom; 2.54mm keepout")
+    (tags marker)
+    (attr virtual)
+    (fp_text reference REF** (at 3.4 0.7) (layer F.SilkS) hide
+      (effects (font (size 1 1) (thickness 0.15)))
+    )
+    (fp_text value Fiducial_1mm_Dia_2.54mm_Outer_CopperBottom (at 0 -1.8) (layer F.Fab)
+      (effects (font (size 1 1) (thickness 0.15)))
+    )
+    (fp_circle (center 0 0) (end 1.55 0) (layer B.CrtYd) (width 0.05))
+    (pad ~ smd circle (at 0 0) (size 1 1) (layers B.Cu B.Mask)
+      (solder_mask_margin 0.77) (clearance 0.77))
+  )
+  (module Fiducials:Fiducial_1mm_Dia_2.54mm_Outer_CopperBottom (layer F.Cu)
+    (at 41.529 109.728)
+    (descr "Circular Fiducial, 1mm bare copper bottom; 2.54mm keepout")
+    (tags marker)
+    (attr virtual)
+    (fp_text reference REF** (at 3.4 0.7) (layer F.SilkS) hide
+      (effects (font (size 1 1) (thickness 0.15)))
+    )
+    (fp_text value Fiducial_1mm_Dia_2.54mm_Outer_CopperBottom (at 0 -1.8) (layer F.Fab)
+      (effects (font (size 1 1) (thickness 0.15)))
+    )
+    (fp_circle (center 0 0) (end 1.55 0) (layer B.CrtYd) (width 0.05))
+    (pad ~ smd circle (at 0 0) (size 1 1) (layers B.Cu B.Mask)
+      (solder_mask_margin 0.77) (clearance 0.77))
+  )
+  (module Fiducials:Fiducial_1mm_Dia_2.54mm_Outer_CopperBottom (layer F.Cu)
+    (at 155.829 110.49)
+    (descr "Circular Fiducial, 1mm bare copper bottom; 2.54mm keepout")
+    (tags marker)
+    (attr virtual)
+    (fp_text reference REF** (at 3.4 0.7) (layer F.SilkS) hide
+      (effects (font (size 1 1) (thickness 0.15)))
+    )
+    (fp_text value Fiducial_1mm_Dia_2.54mm_Outer_CopperBottom (at 0 -1.8) (layer F.Fab)
+      (effects (font (size 1 1) (thickness 0.15)))
+    )
+    (fp_circle (center 0 0) (end 1.55 0) (layer B.CrtYd) (width 0.05))
+    (pad ~ smd circle (at 0 0) (size 1 1) (layers B.Cu B.Mask)
+      (solder_mask_margin 0.77) (clearance 0.77))
+  )
+  (module Fiducials:Fiducial_1mm_Dia_2.54mm_Outer_CopperBottom (layer F.Cu)
+    (at 155.829 49.53)
+    (descr "Circular Fiducial, 1mm bare copper bottom; 2.54mm keepout")
+    (tags marker)
+    (attr virtual)
+    (fp_text reference REF** (at 3.048 -2.794) (layer F.SilkS) hide
+      (effects (font (size 1 1) (thickness 0.15)))
+    )
+    (fp_text value Fiducial_1mm_Dia_2.54mm_Outer_CopperBottom (at 0 -1.8) (layer F.Fab)
+      (effects (font (size 1 1) (thickness 0.15)))
+    )
+    (fp_circle (center 0 0) (end 1.55 0) (layer B.CrtYd) (width 0.05))
+    (pad ~ smd circle (at 0 0) (size 1 1) (layers B.Cu B.Mask)
+      (solder_mask_margin 0.77) (clearance 0.77))
+  )
   (gr_line (start 78.105 57.0484) (end 77.47 57.0484) (layer F.SilkS) (width 0.15))
